File: pcb/soil_sensor/soil_sensor.kicad_pcb (KiCad board)
At the start: 2 copper layers, 16.5 x 67.8 mm, 2 parts, among them J1 Conn_01x02, U1 Capacitive_Soil_Sensor

Commit message: released Rev A
Other:
- board size 16.5 x 67.8 mm -> 23.6 x 67.8 mm
Changed lines of the file:
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@@
       (outputformat 1)
       (mirror false)
-      (drillshape 1)
+      (drillshape 0)
       (scaleselection 1)
-      (outputdirectory "")
+      (outputdirectory "mfg/RevA/")
     )
   )
@@
     (property "Sheetname" "")
     (attr through_hole)
-    (fp_text reference "J1" (at 0 -2.33 90) (layer "F.SilkS")
+    (fp_text reference "J1" (at -0.05 -2.375 180) (layer "F.SilkS")
       (effects (font (size 1 1) (thickness 0.15)))
     )
@@
     )
   )
+  (gr_line (start 163.6 71.6) (end 162.05 69.6) (layer "B.SilkS") (width 0.15))
+  (gr_line (start 166.825 70.4) (end 166.25 69.6) (layer "B.SilkS") (width 0.15))
+  (gr_line (start 165.8 71.6) (end 164.25 69.6) (layer "B.SilkS") (width 0.15))
+  (gr_line (start 166.625 71.4) (end 165.25 69.6) (layer "B.SilkS") (width 0.15))
+  (gr_line (start 162.375 71.6) (end 160.825 69.6) (layer "B.SilkS") (width 0.15))
+  (gr_line (start 164.8 71.6) (end 163.25 69.6) (layer "B.SilkS") (width 0.15))
+  (gr_line (start 166.225 71.6) (end 166.8 70.8) (layer "F.SilkS") (width 0.15))
+  (gr_line (start 163.225 71.6) (end 164.775 69.6) (layer "F.SilkS") (width 0.15))
+  (gr_line (start 162.025 71.6) (end 163.575 69.6) (layer "F.SilkS") (width 0.15))
+  (gr_line (start 160.8 71.6) (end 162.35 69.6) (layer "F.SilkS") (width 0.15))
+  (gr_line (start 164.225 71.6) (end 165.775 69.6) (layer "F.SilkS") (width 0.15))
+  (gr_line (start 165.225 71.6) (end 166.6 69.8) (layer "F.SilkS") (width 0.15))
+  (gr_line (start 166.1 72) (end 161 72) (layer "Edge.Cuts") (width 0.1))
   (gr_line (start 144.5 72) (end 147.5 72) (layer "Edge.Cuts") (width 0.1))
-  (gr_arc (start 159 72) (mid 159.707107 72.292893) (end 160 73) (layer "Edge.Cuts") (width 0.1))
+  (gr_arc (start 160 73) (mid 160.292893 72.292893) (end 161 72) (layer "Edge.Cuts") (width 0.1))
   (gr_arc (start 160 128.75) (mid 151.75 137) (end 143.5 128.75) (layer "Edge.Cuts") (width 0.1))
   (gr_line (start 160 73) (end 160 128.75) (layer "Edge.Cuts") (width 0.1))
-  (gr_line (start 156 72) (end 159 72) (layer "Edge.Cuts") (width 0.1))
   (gr_line (start 143.5 73) (end 143.5 128.75) (layer "Edge.Cuts") (width 0.1))
-  (gr_arc (start 156 72) (mid 155.292893 71.707107) (end 155 71) (layer "Edge.Cuts") (width 0.1))
-  (gr_arc (start 154 69.25) (mid 154.707107 69.542893) (end 155 70.25) (layer "Edge.Cuts") (width 0.1))
-  (gr_line (start 154 69.25) (end 149.5 69.25) (layer "Edge.Cuts") (width 0.1))
-  (gr_line (start 155 70.25) (end 155 71) (layer "Edge.Cuts") (width 0.1))
+  (gr_arc (start 167.092893 71.057107) (mid 166.798893 71.741736) (end 166.1 72) (layer "Edge.Cuts") (width 0.1))
+  (gr_arc (start 166 69.25) (mid 166.770552 69.546861) (end 167.092893 70.307107) (layer "Edge.Cuts") (width 0.1))
+  (gr_line (start 166 69.25) (end 149.5 69.25) (layer "Edge.Cuts") (width 0.1))
+  (gr_line (start 167.092893 70.307107) (end 167.092893 71.057107) (layer "Edge.Cuts") (width 0.1))
   (gr_arc (start 148.5 70.25) (mid 148.792893 69.542893) (end 149.5 69.25) (layer "Edge.Cuts") (width 0.1))
   (gr_arc (start 143.5 73) (mid 143.792893 72.292893) (end 144.5 72) (layer "Edge.Cuts") (width 0.1))
