File: pcb/flora/sensor.kicad_sch (KiCad schematic)
At the start: 4 parts, among them IC2 SHT20

Commit message: added image
Other:
- title: (none) -> FLORA
Changed lines of the file:
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@@
 (kicad_sch (version 20211123) (generator eeschema)
   (paper "A3")
+  (title_block
+    (title "FLORA")
+    (date "2022-06-01")
+    (rev "B")
+  )
   (junction (at 109.855 76.835) (diameter 0) (color 0 0 0 0)
   )

Commit message: Finished schematic for RA-01 design
Other:
- title: FLORA -> FLORA-RA01H
Changed lines of the file:
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@@
   (paper "A3")
   (title_block
-    (title "FLORA")
-    (date "2022-07-01")
+    (title "FLORA-RA01H")
+    (date "2022-12-05")
     (rev "C")
   )
