File: pcb/flora/usb.kicad_sch (KiCad schematic)
At the start: 8 parts, among them J6 Conn_01x04, U4 CH340B

Commit message: added image
Parts:
- U4: value CH340B -> CH340C; symbol Misc_JLC:CH340B -> Misc_JLC:CH340C; LCSC C81010 -> C84681
Other:
- title: (none) -> FLORA
Changed lines of the file:
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@@
 (kicad_sch (version 20211123) (generator eeschema)
   (paper "A3")
+  (title_block
+    (title "FLORA")
+    (date "2022-06-01")
+    (rev "B")
+  )
   (junction (at 193.675 78.74) (diameter 0) (color 0 0 0 0)
   )
@@
     (pin "4")
   )
-  (symbol (lib_id "Misc_JLC:CH340B") (at 177.165 97.155 0) (unit 1)
+  (symbol (lib_id "Misc_JLC:CH340C") (at 177.165 97.155 0) (unit 1)
     (in_bom yes) (on_board yes) (fields_autoplaced)
     (property "Reference" "U4" (id 0) (at 179.1844 112.0045 0)
       (effects (font (size 1.27 1.27)) (justify left))
     )
-    (property "Value" "CH340B" (id 1) (at 179.1844 114.7796 0)
+    (property "Value" "CH340C" (id 1) (at 179.1844 114.7796 0)
       (effects (font (size 1.27 1.27)) (justify left))
     )
@@
       (effects (font (size 1.27 1.27)) hide)
     )
-    (property "LCSC" "C81010" (id 4) (at 210.9978 107.2642 0)
-      (effects (font (size 1.27 1.27)) hide)
-    )
+    (property "LCSC" "C84681" (id 4) (at 210.9978 107.2642 0)
+      (effects (font (size 1.27 1.27)) hide)
+    )

Commit message: Finished schematic for RA-01 design
Other:
- title: FLORA -> FLORA-RA01H
Changed lines of the file:
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@@
   (paper "A3")
   (title_block
-    (title "FLORA")
-    (date "2022-07-01")
+    (title "FLORA-RA01H")
+    (date "2022-12-05")
     (rev "C")
   )
