File: pcb/flora/flora.kicad_sch (KiCad schematic)
At the start: 4 parts

Commit message: released Rev A
Connections:
- no-connect marks 0 -> 4
Changed lines of the file:
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@@
     (rev "A")
   )
+  (no_connect (at 200.66 109.855))
+  (no_connect (at 200.66 104.14))
+  (no_connect (at 200.66 106.045))
+  (no_connect (at 200.66 107.95))
   (wire (pts (xy 227.33 93.98) (xy 248.285 93.98))
     (stroke (width 0) (type default) (color 0 0 0 0))
@@
     (stroke (width 0) (type default) (color 0 0 0 0))
   )
+  (wire (pts (xy 200.66 107.95) (xy 201.93 107.95))
+    (stroke (width 0) (type default) (color 0 0 0 0))
+  )
   (wire (pts (xy 169.545 118.11) (xy 201.93 118.11))
     (stroke (width 0) (type default) (color 0 0 0 0))
@@
     (stroke (width 0) (type default) (color 0 0 0 0))
   )
+  (wire (pts (xy 200.66 104.14) (xy 201.93 104.14))
+    (stroke (width 0) (type default) (color 0 0 0 0))
+  )
   (wire (pts (xy 227.33 107.315) (xy 248.285 107.315))
     (stroke (width 0) (type default) (color 0 0 0 0))
@@
     (stroke (width 0) (type default) (color 0 0 0 0))
   )
+  (wire (pts (xy 200.66 109.855) (xy 201.93 109.855))
+    (stroke (width 0) (type default) (color 0 0 0 0))
+  )
   (wire (pts (xy 186.055 98.425) (xy 201.93 98.425))
+    (stroke (width 0) (type default) (color 0 0 0 0))
+  )
+  (wire (pts (xy 200.66 106.045) (xy 201.93 106.045))
     (stroke (width 0) (type default) (color 0 0 0 0))
   )
@@
       (reference "IC6") (unit 1) (value "TPS54331DR") (footprint "SOIC127P600X175-8N")
     )
+    (path "/99e49cb0-f4b5-4d70-9f27-821a65e53a72/1b89367c-4aae-4e6b-b570-3f6f87660807"
+      (reference "IC7") (unit 1) (value "AMS1117-3.3") (footprint "Package_TO_SOT_SMD:SOT-223-3_TabPin2")
+    )
     (path "/74a12308-4a41-4350-a047-fe690f0632a6/55a5862a-10a4-4102-a2c3-317b201915d7"
       (reference "J1") (unit 1) (value "KF350-3.5-2P") (footprint "KF350352P")
@@
       (reference "U1") (unit 1) (value "Ai-Thinker-Ra-01") (footprint "RF_Module:Ai-Thinker-Ra-01-LoRa")
     )
-    (path "/99e49cb0-f4b5-4d70-9f27-821a65e53a72/8bb93efb-f20a-4989-8e16-adcb4d6687f1"
-      (reference "U2") (unit 1) (value "AMS1117") (footprint "Package_TO_SOT_SMD:SOT-223-3_TabPin2")
-    )
     (path "/74a12308-4a41-4350-a047-fe690f0632a6/d0a49961-7295-411a-ad35-86faadb61ab4"

Commit message: Finished schematic for RA-01 design
Connections:
- no-connect marks 4 -> 0
Other:
- sheet LoRa ports: added none; removed BUSY, DIO1, DIO2, DIO3, RXEN
- sheet Microcontroller ports: added none; removed BUSY, DIO1, DIO2, DIO3, RXEN, TCK, TDI, TDO, TMS
- title: FLORA -> FLORA-RA01H
