File: pcb/flora/connector.kicad_sch (KiCad schematic)
At the start: 9 parts, among them J1 KF350-3.5-2P, J2 KF350-3.5-2P, J3 KF350-3.5-2P, J4 10118193-0001LF, J5 PH-2V, U3 USBLC6-2P6

Commit message: released Rev A
Other:
- moved on the sheet: C21, D4, J1, J2, J3, J4, J5, TP3, U3

Commit message: added image
Other:
- title: (none) -> FLORA
Changed lines of the file:
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@@
 (kicad_sch (version 20211123) (generator eeschema)
   (paper "A3")
+  (title_block
+    (title "FLORA")
+    (date "2022-06-01")
+    (rev "B")
+  )
   (junction (at 123.825 116.84) (diameter 0) (color 0 0 0 0)
   )

Commit message: Finished schematic for RA-01 design
Other:
- title: FLORA -> FLORA-RA01H
Changed lines of the file:
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@@
   (paper "A3")
   (title_block
-    (title "FLORA")
-    (date "2022-07-01")
+    (title "FLORA-RA01H")
+    (date "2022-12-05")
     (rev "C")
   )

Commit message: finished smps layout
Parts:
- removed TP3: USB Test Point, personal:USB_TestPoint, symbol personal:USB Test Point
Changed lines of the file:
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@@
     (rev "C")
   )
-  (junction (at 123.825 116.84) (diameter 0) (color 0 0 0 0)
-  )
   (junction (at 179.705 111.125) (diameter 0) (color 0 0 0 0)
   )
-  (junction (at 118.745 124.46) (diameter 0) (color 0 0 0 0)
-  )
-  (junction (at 121.285 119.38) (diameter 0) (color 0 0 0 0)
-  )
   (junction (at 137.16 146.05) (diameter 0) (color 0 0 0 0)
   )
   (junction (at 140.335 111.125) (diameter 0) (color 0 0 0 0)
-  )
-  (junction (at 126.365 114.3) (diameter 0) (color 0 0 0 0)
   )
   (no_connect (at 88.9 121.92))
@@
   (no_connect (at 88.9 119.38))
   (no_connect (at 88.9 116.84))
-  (wire (pts (xy 114.3 116.84) (xy 123.825 116.84))
-    (stroke (width 0) (type default) (color 0 0 0 0))
-  )
-  (wire (pts (xy 126.365 114.3) (xy 140.335 114.3))
-    (stroke (width 0) (type default) (color 0 0 0 0))
-  )
   (polyline (pts (xy 316.865 108.585) (xy 316.865 139.065))
     (stroke (width 0) (type default) (color 0 0 0 0))
@@
     (stroke (width 0) (type default) (color 0 0 0 0))
   )
-  (wire (pts (xy 121.285 100.33) (xy 121.285 119.38))
-    (stroke (width 0) (type default) (color 0 0 0 0))
-  )
   (wire (pts (xy 102.235 212.725) (xy 95.885 212.725))
     (stroke (width 0) (type default) (color 0 0 0 0))
@@
     (stroke (width 0) (type default) (color 0 0 0 0))
   )
-  (wire (pts (xy 114.3 114.3) (xy 126.365 114.3))
+  (wire (pts (xy 114.3 114.3) (xy 140.335 114.3))
     (stroke (width 0) (type default) (color 0 0 0 0))
   )
@@
     (stroke (width 0) (type default) (color 0 0 0 0))
   )
-  (wire (pts (xy 114.3 124.46) (xy 118.745 124.46))
-    (stroke (width 0) (type default) (color 0 0 0 0))
-  )
-  (wire (pts (xy 123.825 116.84) (xy 167.005 116.84))
+  (wire (pts (xy 114.3 116.84) (xy 167.005 116.84))
     (stroke (width 0) (type default) (color 0 0 0 0))
   )
@@
     (stroke (width 0) (type default) (color 0 0 0 0))
   )
-  (wire (pts (xy 118.745 102.87) (xy 118.745 124.46))
-    (stroke (width 0) (type default) (color 0 0 0 0))
-  )
   (wire (pts (xy 137.16 124.46) (xy 137.16 146.05))
     (stroke (width 0) (type default) (color 0 0 0 0))
   )
-  (wire (pts (xy 118.745 124.46) (xy 137.16 124.46))
+  (wire (pts (xy 114.3 124.46) (xy 137.16 124.46))
     (stroke (width 0) (type default) (color 0 0 0 0))
   )
@@
     (stroke (width 0) (type default) (color 0 0 0 0))
   )
-  (wire (pts (xy 114.3 119.38) (xy 121.285 119.38))
-    (stroke (width 0) (type default) (color 0 0 0 0))
-  )
-  (wire (pts (xy 126.365 95.25) (xy 126.365 114.3))
+  (wire (pts (xy 114.3 119.38) (xy 167.005 119.38))
     (stroke (width 0) (type default) (color 0 0 0 0))
   )
@@
     (stroke (width 0) (type default) (color 0 0 0 0))
   )
-  (wire (pts (xy 121.285 119.38) (xy 167.005 119.38))
-    (stroke (width 0) (type default) (color 0 0 0 0))
-  )
-  (wire (pts (xy 105.41 102.87) (xy 118.745 102.87))
-    (stroke (width 0) (type default) (color 0 0 0 0))
-  )
   (wire (pts (xy 179.705 107.95) (xy 179.705 111.125))
     (stroke (width 0) (type default) (color 0 0 0 0))
   )
-  (wire (pts (xy 105.41 95.25) (xy 126.365 95.25))
-    (stroke (width 0) (type default) (color 0 0 0 0))
-  )
-  (wire (pts (xy 105.41 100.33) (xy 121.285 100.33))
-    (stroke (width 0) (type default) (color 0 0 0 0))
-  )
   (polyline (pts (xy 193.675 160.909) (xy 78.105 160.909))
     (stroke (width 0) (type default) (color 0 0 0 0))
@@
     (stroke (width 0) (type default) (color 0 0 0 0))
   )
-  (wire (pts (xy 105.41 97.79) (xy 123.825 97.79))
-    (stroke (width 0) (type default) (color 0 0 0 0))
-  )
   (wire (pts (xy 95.885 198.12) (xy 102.235 198.12))
     (stroke (width 0) (type default) (color 0 0 0 0))
   )
   (polyline (pts (xy 200.025 146.177) (xy 200.025 95.885))
-    (stroke (width 0) (type default) (color 0 0 0 0))
-  )
-  (wire (pts (xy 123.825 97.79) (xy 123.825 116.84))
     (stroke (width 0) (type default) (color 0 0 0 0))
   )
@@
     (pin "1")
   )
-  (symbol (lib_id "personal:USB Test Point") (at 105.41 95.25 0) (mirror y) (unit 1)
-    (in_bom yes) (on_board yes) (fields_autoplaced)
-    (property "Reference" "TP3" (id 0) (at 96.52 88.7943 0))
-    (property "Value" "USB Test Point" (id 1) (at 96.52 91.5694 0))
-    (property "Footprint" "personal:USB_TestPoint" (id 2) (at 83.82 92.71 0)
-      (effects (font (size 1.27 1.27)) (justify left) hide)
-    )
-    (property "Datasheet" "" (id 3) (at 83.82 95.25 0)
-      (effects (font (size 1.27 1.27)) (justify left) hide)
-    )
-    (property "Description" "USB Test Point" (id 4) (at 83.82 97.79 0)
-      (effects (font (size 1.27 1.27)) (justify left) hide)
-    )
-    (pin "1")
-    (pin "2")
-    (pin "3")
-    (pin "4")
-  )
   (symbol (lib_id "Connector_JLC:KF350-3.5-2P") (at 102.235 198.12 0) (unit 1)
