File: pcb/flora/flora.kicad_pcb (KiCad board)
At the start: 4 copper layers, 59 x 59 mm, 94 parts, among them IC1 ESP32-WROOM-32E(8MB), IC2 SHT20, IC3 TP4056X, IC4 FS8205A, IC5 DW01+G, IC6 TPS54331DR, J1 KF350-3.5-2P, J2 KF350-3.5-2P, J3 KF350-3.5-2P, J4 10118193-0001LF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

Commit message: released Rev A
Connections:
- J1 pad 1: GPIO34 -> GPIO14
- J2 pad 1: GPIO35 -> GPIO12
- J3 pad 1: GPIO33 -> GPIO13
Routing:
- net GPIO35: track 59.4 -> 0.00 mm, vias 2 -> 0
- net GPIO12: track 14.2 -> 71.0 mm, vias 0 -> 2
- net GPIO33: track 54.1 -> 0.00 mm, vias 2 -> 0
- net GPIO34: track 52.2 -> 0.00 mm, vias 2 -> 0
- net GPIO13: track 17.2 -> 66.0 mm, vias 2 -> 4
- net GPIO14: track 37.2 -> 85.8 mm, vias 2 -> 4

Commit message: added image
Parts:
- removed J8: Conn_01x04, Connector_PinHeader_1.27mm:PinHeader_1x04_P1.27mm_Vertical
- removed U2: AMS1117, Package_TO_SOT_SMD:SOT-223-3_TabPin2
- added C26: 220uF_E_LV, Capacitor_SMD:CP_Elec_6.3x5.4, F.Cu at (219.3, 112.3)
- added IC7: AMS1117-3.3, Package_TO_SOT_SMD:SOT-223-3_TabPin2, F.Cu at (223.5, 137.8)
- U1: value Ai-Thinker-Ra-01 -> Ai-Thinker-Ra-01H
- U4: value CH340B -> CH340C
- moved C20 16.3 mm to (216.9, 131.0), turned to -90 degrees
- moved C18 15.0 mm to (227.8, 121.6), turned to 180 degrees
- moved C19 14.8 mm to (216.8, 128.1), turned to 180 degrees
- moved R6 14.3 mm to (229.7, 108.4), turned to 180 degrees
- moved JP6 13.4 mm to (220.0, 130.1), turned to -90 degrees
- moved C8 13.0 mm to (231.8, 120.0), turned to 0 degrees
- moved C10 12.8 mm to (227.0, 120.0), turned to 180 degrees
- moved C5 12.7 mm to (229.7, 111.4)
- moved C7 12.7 mm to (230.1, 109.9), turned to 90 degrees
- moved R11 12.1 mm to (229.5, 120.0), turned to 0 degrees
- moved C14 10.5 mm to (216.8, 126.0), turned to 180 degrees
- moved R10 9.07 mm to (231.7, 111.4), turned to 0 degrees
- moved L1 8.95 mm to (225.8, 109.5), turned to 180 degrees
- moved R12 8.56 mm to (231.2, 109.9)
- moved R9 8.55 mm to (231.2, 107.9)
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Connections:
- C7 pad 1: Net-(C7-Pad1) -> Net-(C5-Pad1)
- C7 pad 2: GND -> Net-(C7-Pad2)
- R6 pad 1: Net-(C5-Pad1) -> Net-(C7-Pad2)
- R6 pad 2: Net-(C7-Pad1) -> GND
Routing:
- net Net-(C14-Pad1): track 12.0 -> 40.6 mm, vias 0 -> 2
- net GPIO15: track 25.3 -> 0.00 mm, vias 2 -> 0
- net +3V3: track 68.4 -> 49.4 mm, vias 11 -> 10
- net GPIO13: track 66.0 -> 48.2 mm, vias 4 -> 2
- net GPIO12: track 71.0 -> 56.8 mm
- net VDD: track 139.5 -> 152.6 mm
- net Net-(C5-Pad1): track 15.3 -> 2.38 mm
- net GPIO14: track 85.8 -> 74.5 mm
- net Net-(C10-Pad2): track 25.4 -> 14.4 mm
- net Net-(IC6-Pad5): track 9.80 -> 2.45 mm
- net GND: track 113.3 -> 106.5 mm, vias 32 -> 76
- net Net-(C7-Pad1): track 0.96 -> 0.00 mm
- net Net-(C7-Pad2): track 0.00 -> 0.92 mm
- added copper zone on B.Cu, net GND
- removed copper zone on F.Cu, net Net-(C14-Pad1)
Other:
- board text added: "elektroThing FLORA Rev B June 2022"

Commit message: Replaced SMPS
Parts:
- removed C18: 22u, Capacitor_SMD:C_0805_2012Metric
- removed C26: 220uF_E_LV, Capacitor_SMD:CP_Elec_6.3x5.4
- removed D3: B340A-13-F, SamacSys_Parts:DIOM5226X240N
- removed R10: 3.3k, Resistor_SMD:R_0402_1005Metric
- removed R11: 10k, Resistor_SMD:R_0402_1005Metric
- removed R12: 220, Resistor_SMD:R_0402_1005Metric
- C14: value 10u -> 22u
- C5: value 4.7n -> 10u; footprint Capacitor_SMD:C_0402_1005Metric -> Capacitor_SMD:C_0805_2012Metric
- C7: value 8.2n -> 10u; footprint Capacitor_SMD:C_0402_1005Metric -> Capacitor_SMD:C_0805_2012Metric
- C8: value 8.2n -> 68p
- IC6: value TPS54331DR -> TPS54302DDCR; footprint SamacSys_Parts:SOIC127P600X175-8N -> SamacSys_Parts:SOT95P280X110-6N
- L1: value 10uH -> 5.6uH
- R6: value 1k -> 100k
- R9: value 10k -> 22k
- moved C20 16.6 mm to (227.3, 118.0), turned to 180 degrees
- moved C8 15.7 mm to (218.4, 111.9), turned to 90 degrees
- moved R9 14.4 mm to (217.9, 113.4), turned to 0 degrees
- moved C19 13.2 mm to (227.3, 120.1)
- moved R6 12.8 mm to (217.4, 111.9), turned to 90 degrees
- moved C14 11.2 mm to (227.3, 122.2)
- moved IC6 8.93 mm to (221.1, 112.4), turned to 180 degrees
- moved C10 8.37 mm to (220.4, 114.8), turned to 0 degrees
- moved L1 6.16 mm to (229.9, 114.1), turned to -90 degrees
- moved C5 5.39 mm to (224.4, 112.4), turned to -90 degrees
- moved C7 4.38 mm to (226.5, 112.4), turned to -90 degrees
Connections:
- C14 pad 1: Net-(C14-Pad1) -> Net-(C19-Pad1)
- C19 pad 1: Net-(C14-Pad1) -> Net-(C19-Pad1)
- C20 pad 1: Net-(C14-Pad1) -> Net-(C19-Pad1)
- C5 pad 1: Net-(C5-Pad1) -> VDD
- C7 pad 1: Net-(C5-Pad1) -> VDD
- C7 pad 2: Net-(C7-Pad2) -> GND
- C8 pad 1: Net-(C8-Pad1) -> Net-(C19-Pad1)
- C8 pad 2: GND -> Net-(C8-Pad2)
- IC6 pad 1: Net-(C10-Pad1) -> GND
- IC6 pad 2: VDD -> Net-(C10-Pad2)
- IC6 pad 3: Net-(IC6-Pad3) -> VDD
- IC6 pad 4: Net-(C8-Pad1) -> Net-(C8-Pad2)
- IC6 pad 5: Net-(IC6-Pad5) -> unconnected-(IC6-Pad5)
- IC6 pad 6: Net-(C5-Pad1) -> Net-(C10-Pad1)
- JP6 pad 1: Net-(C14-Pad1) -> Net-(C19-Pad1)
- L1 pad 2: Net-(C14-Pad1) -> Net-(C19-Pad1)
- R6 pad 1: Net-(C7-Pad2) -> Net-(C19-Pad1)
- R6 pad 2: GND -> Net-(C8-Pad2)
- R9 pad 1: Net-(C14-Pad1) -> Net-(C8-Pad2)
- R9 pad 2: Net-(R12-Pad1) -> GND
Routing:
- net Net-(C14-Pad1): track 40.6 -> 0.00 mm, vias 2 -> 0
- net Net-(C19-Pad1): track 0.00 -> 33.2 mm, vias 0 -> 2
- net GND: track 106.5 -> 90.9 mm, vias 76 -> 28
- net Net-(C8-Pad2): track 0.00 -> 5.70 mm
- net VDD: track 152.6 -> 149.7 mm
- net Net-(IC6-Pad5): track 2.45 -> 0.00 mm
- net Net-(C5-Pad1): track 2.38 -> 0.00 mm
- net Net-(C10-Pad2): track 14.4 -> 15.9 mm, vias 2 -> 7
- net Net-(C8-Pad1): track 1.57 -> 0.00 mm
- net Net-(IC6-Pad3): track 1.56 -> 0.00 mm
- net Net-(R12-Pad1): track 0.98 -> 0.00 mm
- net Net-(C7-Pad2): track 0.92 -> 0.00 mm
- added copper zone on B.Cu, net Net-(C10-Pad2)
- added copper zone on F.Cu, net Net-(C19-Pad1)
- added copper zone on F.Cu, net VDD
- removed copper zone on B.Cu, net GND

Commit message: Finished schematic for RA-01 design
Parts:
- removed C14, C19, C20: 22u, Capacitor_SMD:C_0805_2012Metric
- removed JP1, JP2, JP3, JP4, JP5, JP6: SB_NO, Jumper:SolderJumper-2_P1.3mm_Open_TrianglePad1.0x1.5mm
- added J7: U.FL-R-SMT-1_10_, SamacSys_Parts:U.FL-R-SMT-1_10_, F.Cu at (193.0, 116.7)
- added R10: 1M, Resistor_SMD:R_0402_1005Metric, F.Cu at (253.3, 121.5)
- C10: value 100n -> 10u; footprint Capacitor_SMD:C_0402_1005Metric -> Capacitor_SMD:C_0805_2012Metric
- C7: value 10u -> 1n; footprint Capacitor_SMD:C_0805_2012Metric -> Capacitor_SMD:C_0402_1005Metric
- C8: value 68p -> 10u; footprint Capacitor_SMD:C_0402_1005Metric -> Capacitor_SMD:C_0805_2012Metric
- IC6: value TPS54302DDCR -> TPS63051RMWR; footprint SamacSys_Parts:SOT95P280X110-6N -> SamacSys_Parts:QFN50P250X250X100-12N-D
- IC7: value AMS1117-3.3 -> XC6227C331MR-G; footprint Package_TO_SOT_SMD:SOT-223-3_TabPin2 -> SamacSys_Parts:SOT95P280X130-5N
- L1: value 5.6uH -> LVF201B12-1R5M-N; footprint SamacSys_Parts:INDPM4040X300N -> SamacSys_Parts:LVF201B121R5MN
- R1: value 0 -> DNF_0805
- R6: value 100k -> 560k; footprint Resistor_SMD:R_0402_1005Metric -> Resistor_SMD:R_0603_1608Metric
- R9: value 22k -> 180k
- moved R2 64.5 mm to (254.2, 116.1), turned to 0 degrees
- moved R9 40.2 mm to (257.7, 118.6)
- moved C5 34.6 mm to (258.8, 116.1), turned to 0 degrees
- moved R6 34.1 mm to (249.4, 123.7), turned to 0 degrees
- moved C10 33.9 mm to (254.1, 119.0)
- moved C8 32.5 mm to (249.6, 120.9), turned to 0 degrees
- moved C7 31.0 mm to (256.2, 121.5), turned to 0 degrees
- moved IC6 28.7 mm to (249.4, 117.0), turned to 0 degrees
- moved IC7 26.2 mm to (244.8, 122.4), turned to 0 degrees
- moved L1 15.0 mm to (244.6, 117.3), turned to 0 degrees
- moved R1 0.51 mm to (195.3, 120.9)
Connections:
- C10 pad 1: Net-(C10-Pad1) -> +3V3
- C10 pad 2: Net-(C10-Pad2) -> GND
- C7 pad 1: VDD -> Net-(C7-Pad1)
- C8 pad 1: Net-(C14-Pad1) -> +3V3
- C8 pad 2: Net-(C8-Pad2) -> GND
- IC6 pad 1: GND -> Net-(IC6-Pad1)
- IC6 pad 2: Net-(C10-Pad2) -> GND
- IC6 pad 3: VDD -> Net-(IC6-Pad3)
- IC6 pad 4: Net-(C8-Pad2) -> +3V3
- IC6 pad 5: unconnected-(IC6-Pad5) -> Net-(IC6-Pad5)
- IC6 pad 6: Net-(C10-Pad1) -> GND
- IC7 pad 1: GND -> VDD
- IC7 pad 2: Net-(IC7-Pad2) -> GND
- JP7 pad 1: Net-(IC7-Pad2) -> Net-(JP7-Pad1)
- L1 pad 1: Net-(C10-Pad2) -> Net-(IC6-Pad1)
- L1 pad 2: Net-(C14-Pad1) -> Net-(IC6-Pad3)
- R2 pad 1: Net-(R2-Pad1) -> VDD
- R2 pad 2: GPIO2 -> Net-(IC6-Pad10)
- R6 pad 1: Net-(C14-Pad1) -> +3V3
- R6 pad 2: Net-(C8-Pad2) -> Net-(IC6-Pad5)
- R9 pad 1: Net-(C8-Pad2) -> Net-(IC6-Pad5)
- U1 pad 10: Net-(JP4-Pad1) -> unconnected-(U1-Pad10)
- U1 pad 11: Net-(JP5-Pad1) -> unconnected-(U1-Pad11)
- U1 pad 5: Net-(R2-Pad1) -> GPIO2
- U1 pad 6: Net-(JP1-Pad1) -> unconnected-(U1-Pad6)
- U1 pad 7: Net-(JP2-Pad1) -> unconnected-(U1-Pad7)
- U1 pad 8: Net-(JP3-Pad1) -> unconnected-(U1-Pad8)
Routing:
- net GPIO12: track 56.8 -> 0.00 mm, vias 2 -> 0
- net GPIO14: track 74.5 -> 26.0 mm, vias 4 -> 2
- net GPIO13: track 48.2 -> 0.00 mm, vias 2 -> 0
- net GPIO21: track 37.2 -> 0.00 mm, vias 2 -> 0
- net GPIO25: track 35.1 -> 0.00 mm, vias 2 -> 0
- net GPIO26: track 34.8 -> 0.00 mm, vias 2 -> 0
- net VDD: track 149.7 -> 115.7 mm, vias 6 -> 5
- net Net-(C14-Pad1): track 33.2 -> 0.00 mm, vias 2 -> 0
- net GPIO22: track 31.9 -> 0.00 mm, vias 2 -> 0
- net Net-(JP5-Pad1): track 30.0 -> 0.00 mm, vias 2 -> 0
- net GPIO27: track 28.6 -> 0.00 mm, vias 2 -> 0
- net Net-(JP4-Pad1): track 26.3 -> 0.00 mm, vias 2 -> 0
- net GPIO2: track 17.9 -> 0.00 mm
- net Net-(C10-Pad2): track 15.9 -> 0.00 mm, vias 7 -> 0
- net +3V3: track 49.4 -> 37.5 mm
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- removed copper zone on B.Cu, net Net-(C10-Pad2)
- removed copper zone on F.Cu, net Net-(C14-Pad1)
- removed copper zone on B.Cu, net Net-(IC7-Pad2)
- removed copper zone on F.Cu, net Net-(IC7-Pad2)
- removed copper zone on F.Cu, net VDD
Other:
- board text removed: "elektroThing FLORA Rev B June 2022"

Commit message: base placement completed
Parts:
- removed JP7: SB_NC, Jumper:SolderJumper-2_P1.3mm_Bridged_Pad1.0x1.5mm
- added R11: DNF_0805, Resistor_SMD:R_0805_2012Metric_Pad1.20x1.40mm_HandSolder, F.Cu at (219.9, 127.0)
- added R12: 0, Resistor_SMD:R_0805_2012Metric_Pad1.20x1.40mm_HandSolder, F.Cu at (219.9, 130.9)
- moved C5 32.1 mm to (227.2, 110.4)
- moved C10 30.7 mm to (223.4, 120.8)
- moved R9 30.4 mm to (227.3, 118.6), turned to -90 degrees
- moved C7 28.7 mm to (228.1, 115.8), turned to 90 degrees
- moved R2 27.1 mm to (227.3, 112.5)
- moved C8 26.3 mm to (223.4, 123.0)
- moved R6 24.7 mm to (225.2, 118.4)
- moved R10 24.7 mm to (229.1, 116.7), turned to 90 degrees
- moved IC7 24.2 mm to (224.7, 135.9)
- moved IC6 23.9 mm to (225.6, 115.6)
- moved L1 22.9 mm to (221.7, 115.7), turned to 180 degrees
- moved C13 8.02 mm to (221.5, 135.8), turned to -90 degrees
Connections:
- C10 pad 1: +3V3 -> Net-(C10-Pad1)
- C15 pad 1: +3V3 -> Net-(IC7-Pad5)
- C8 pad 1: +3V3 -> Net-(C10-Pad1)
- IC6 pad 4: +3V3 -> Net-(C10-Pad1)
- IC7 pad 5: Net-(JP7-Pad1) -> Net-(IC7-Pad5)
- R10 pad 1: +3V3 -> Net-(C10-Pad1)
- R6 pad 1: +3V3 -> Net-(C10-Pad1)
Routing:
- net +3V3: track 37.5 -> 28.8 mm, vias 10 -> 9
- net Net-(IC7-Pad5): track 0.00 -> 1.44 mm, vias 0 -> 1

Commit message: finished smps layout
Parts:
- removed C15: 10u, Capacitor_SMD:C_0805_2012Metric
- removed TP3: USB Test Point, personal:USB_TestPoint
- added C14: 10u_0402, Capacitor_SMD:C_0402_1005Metric, F.Cu at (219.9, 138.1)
- C13: value 10u -> 10u_0402; footprint Capacitor_SMD:C_0805_2012Metric -> Capacitor_SMD:C_0402_1005Metric
- moved R11 8.56 mm to (225.1, 133.8), turned to 0 degrees
- moved R9 8.52 mm to (228.7, 110.2), turned to 180 degrees
- moved C13 8.25 mm to (220.4, 143.9), turned to 90 degrees
- moved C10 7.72 mm to (230.4, 117.6), turned to -90 degrees
- moved R12 7.72 mm to (225.1, 136.6), turned to 0 degrees
- moved C5 7.56 mm to (223.9, 117.2)
- moved C8 7.10 mm to (227.5, 117.2), turned to 180 degrees
- moved R6 7.05 mm to (228.7, 112.3), turned to 90 degrees
- moved IC7 6.58 mm to (220.4, 140.8), turned to 90 degrees
- moved L1 5.76 mm to (225.3, 120.2), turned to -90 degrees
- moved C7 5.08 mm to (227.2, 110.8)
- moved R2 4.05 mm to (224.2, 109.9), turned to -90 degrees
- moved R10 4.00 mm to (230.0, 112.8)
- moved IC6 1.90 mm to (225.7, 113.7), turned to 90 degrees
Routing:
- net +3V3: track 28.8 -> 184.9 mm, vias 9 -> 11
- net Net-(C8-Pad1): track 0.00 -> 33.4 mm
- net VDD: track 115.7 -> 146.1 mm, vias 5 -> 6
- net Net-(J7-Pad3): track 0.00 -> 7.90 mm
- net Net-(IC6-Pad8): track 0.00 -> 6.82 mm, vias 0 -> 2
- net Net-(IC6-Pad3): track 0.00 -> 6.26 mm, vias 0 -> 4
- net Net-(IC6-Pad1): track 0.00 -> 6.22 mm, vias 0 -> 4
- net Net-(IC7-Pad5): track 1.44 -> 7.15 mm, vias 1 -> 0
- net Net-(IC6-Pad5): track 0.00 -> 5.08 mm
- net VBUS: track 16.8 -> 11.8 mm
- net D-: track 16.2 -> 12.1 mm, vias 1 -> 0
- net D+: track 18.4 -> 14.4 mm, vias 1 -> 0
- net EN: track 79.8 -> 75.9 mm
- net Net-(D2-Pad1): track 12.3 -> 9.62 mm
- net Net-(IC6-Pad10): track 0.00 -> 2.02 mm
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- added copper zone on F.Cu, net Net-(C8-Pad1)
- added copper zone on B.Cu, net Net-(IC6-Pad1)
- added copper zone on F.Cu, net Net-(IC6-Pad1)
- added copper zone on B.Cu, net Net-(IC6-Pad3)
- added copper zone on F.Cu, net Net-(IC6-Pad3)
- added copper zone on F.Cu, net VDD
Other:
- board text added: "LDO"
- board text added: "SMPS"
